File: PCB_SRT/PCB_SRT/PCB_SRT.kicad_pcb (KiCad board)
At the start: 2 copper layers, 32 parts, among them U1 Power_header, U2 Stepper_header, U3 ESP32, U4 Stepper_header, U5 RX_TX_header, U6 Encoder_header, U7 Encoder_header, U8 RX_TX_header

Commit message: finish PCB
Parts:
- removed the U1 at (246.0, 147.0)
- removed the U1 at (246.2, 80.1)
- removed the U1 at (36.2, 145.7)
- removed the U2 at (218.1, 143.5)
- removed the U2 at (218.2, 76.5)
- removed the U2 at (39.7, 117.7)
- removed the U3 at (251.2, 58.4)
- removed the U3 at (251.1, 125.4)
- removed the U3 at (57.8, 150.7)
- removed the U4 at (75.3, 127.9)
- removed the U4 at (228.3, 107.9)
- removed the U4 at (228.4, 40.9)
- removed the U5 at (75.0, 107.6)
- removed the U5 at (208.1, 41.2)
- removed the U5 at (207.9, 108.2)
- removed the U6 at (84.2, 120.0)
- removed the U6 at (220.5, 32.1)
- removed the U6 at (220.4, 99.0)
- removed the U7 at (88.0, 120.0)
- removed the U7 at (220.4, 95.2)
- removed the U7 at (155.0, 120.1)
- removed the U7 at (220.5, 28.2)
- removed the U8 at (246.2, 74.5)
- removed the U8 at (246.0, 141.4)
- removed the U8 at (41.8, 145.7)
- added G***: LOGO, LOGO, F.Cu at (244.1, 30.0)
- added G***: LOGO, LOGO, F.Cu at (201.2, 96.8)
- added G***: LOGO, LOGO, F.Cu at (36.6, 109.2)
- added G***: LOGO, LOGO, F.Cu at (201.2, 29.5)
- added G***: LOGO, LOGO, F.Cu at (205.0, 148.2)
- added G***: LOGO, LOGO, F.Cu at (87.4, 148.3)
- added G***: LOGO, LOGO, F.Cu at (154.7, 148.3)
- added G***: LOGO, LOGO, F.Cu at (205.0, 80.8)
- added G***: LOGO, LOGO, F.Cu at (155.2, 105.4)
- added G***: LOGO, LOGO, F.Cu at (87.9, 105.4)
- added G***: LOGO, LOGO, F.Cu at (103.9, 109.2)
- added G***: LOGO, LOGO, F.Cu at (244.1, 97.4)
- added U1: Power_header, Connector_PinHeader_2.54mm:PinHeader_1x02_P2.54mm_Vertical, F.Cu at (35.7, 146.7)
- added U1: Power_header, Connector_PinHeader_2.54mm:PinHeader_1x02_P2.54mm_Vertical, F.Cu at (242.5, 149.0)
- added U1: Power_header, Connector_PinHeader_2.54mm:PinHeader_1x02_P2.54mm_Vertical, F.Cu at (242.5, 81.7)
- added U2: Stepper_header, Connector_PinHeader_2.54mm:PinHeader_1x06_P2.54mm_Vertical, F.Cu at (39.3, 118.7)
- added U2: Stepper_header, Connector_PinHeader_2.54mm:PinHeader_1x06_P2.54mm_Vertical, F.Cu at (214.5, 78.2)
- added U2: Stepper_header, Connector_PinHeader_2.54mm:PinHeader_1x06_P2.54mm_Vertical, F.Cu at (214.5, 145.5)
- added U3: ESP32, project_library:NodeMCU_header, F.Cu at (57.4, 151.7)
- added U3: ESP32, project_library:NodeMCU_header, F.Cu at (247.5, 127.4)
- added U3: ESP32, project_library:NodeMCU_header, F.Cu at (247.5, 60.1)
- added U4: Stepper_header, Connector_PinHeader_2.54mm:PinHeader_1x06_P2.54mm_Vertical, F.Cu at (224.7, 42.6)
- added U4: Stepper_header, Connector_PinHeader_2.54mm:PinHeader_1x06_P2.54mm_Vertical, F.Cu at (74.8, 128.9)
- added U4: Stepper_header, Connector_PinHeader_2.54mm:PinHeader_1x06_P2.54mm_Vertical, F.Cu at (224.7, 109.9)
- added U5: RX_TX_header, Connector_PinHeader_2.54mm:PinHeader_1x03_P2.54mm_Vertical, F.Cu at (74.6, 108.6)
- added U5: RX_TX_header, Connector_PinHeader_2.54mm:PinHeader_1x03_P2.54mm_Vertical, F.Cu at (204.4, 42.9)
- added U5: RX_TX_header, Connector_PinHeader_2.54mm:PinHeader_1x03_P2.54mm_Vertical, F.Cu at (204.4, 110.2)
- added U6: Encoder_header, Connector_PinHeader_2.54mm:PinHeader_1x08_P2.54mm_Vertical, F.Cu at (81.1, 113.4)
- added U6: Encoder_header, Connector_PinHeader_2.54mm:PinHeader_1x08_P2.54mm_Vertical, F.Cu at (209.2, 36.3)
- added U6: Encoder_header, Connector_PinHeader_2.54mm:PinHeader_1x08_P2.54mm_Vertical, F.Cu at (209.2, 103.6)
- added U7: Encoder_header, Connector_PinHeader_2.54mm:PinHeader_1x08_P2.54mm_Vertical, F.Cu at (84.9, 113.4)
- added U7: Encoder_header, Connector_PinHeader_2.54mm:PinHeader_1x08_P2.54mm_Vertical, F.Cu at (152.2, 113.4)
- added U7: Encoder_header, Connector_PinHeader_2.54mm:PinHeader_1x08_P2.54mm_Vertical, F.Cu at (209.2, 32.5)
- added U7: Encoder_header, Connector_PinHeader_2.54mm:PinHeader_1x08_P2.54mm_Vertical, F.Cu at (209.2, 99.8)
- added U8: RX_TX_header, Connector_PinHeader_2.54mm:PinHeader_1x03_P2.54mm_Vertical, F.Cu at (242.5, 76.1)
- added U8: RX_TX_header, Connector_PinHeader_2.54mm:PinHeader_1x03_P2.54mm_Vertical, F.Cu at (242.5, 143.4)
- added U8: RX_TX_header, Connector_PinHeader_2.54mm:PinHeader_1x03_P2.54mm_Vertical, F.Cu at (41.3, 146.7)
- U6: footprint Connector_PinHeader_2.54mm:PinHeader_1x10_P2.54mm_Vertical -> Connector_PinHeader_2.54mm:PinHeader_1x08_P2.54mm_Vertical
- moved U6 7.25 mm to (148.5, 113.4)
- moved U2 0.90 mm to (106.6, 118.7)
- moved U3 0.90 mm to (124.7, 151.7)
- moved U5 0.90 mm to (141.9, 108.6)
- moved U8 0.90 mm to (108.6, 146.7)
- moved U1 0.90 mm to (103.0, 146.7)
- moved U4 0.90 mm to (142.1, 128.9)
Connections:
- U2 pad 4: GND -> Net-(U2-Pad4)
- U2 pad 6: Net-(U2-Pad6) -> GND
- U3 pad 26: Net-(U4-Pad6) -> Net-(U3-Pad26)
- U3 pad 27: Net-(U2-Pad6) -> Net-(U2-Pad5)
- U3 pad 28: Net-(U2-Pad5) -> Net-(U2-Pad4)
- U4 pad 4: GND -> Net-(U3-Pad15)
- U4 pad 5: Net-(U3-Pad15) -> Net-(U3-Pad26)
- U4 pad 6: Net-(U4-Pad6) -> GND
- U6 pad 1: /MISO -> +5V
- U6 pad 3: +5V -> GND
- U6 pad 4: /SCK -> /MISO
- U6 pad 5: GND -> /SCK
- U6 pad 6: GND -> /N_CS_1
Routing:
- net Net-(U3-Pad26): track 0.00 -> 204.7 mm
- net Net-(U4-Pad6): track 196.2 -> 0.00 mm
- net /N_CS_1: track 214.6 -> 281.4 mm
- net /N_CS_2: track 222.8 -> 289.7 mm
- net +5V: track 350.4 -> 391.5 mm
- net Net-(U2-Pad6): track 25.6 -> 0.00 mm
- net Net-(U2-Pad4): track 0.00 -> 21.4 mm
- net /SCK: track 78.1 -> 60.2 mm
- net /MISO: track 70.6 -> 61.6 mm
- net Net-(U3-Pad15): track 23.5 -> 28.2 mm
- net Net-(U2-Pad5): track 25.6 -> 21.4 mm
Other:
- board text added: "Antenna Pointing Mechanism V1"
- board text added: "STEP DIR ENABLE BOOST FAULT GND"
- board text added: "VCC GND GND MISO CLK N_CS GND GND"
- board text removed: "MISO GND 5V SCK GND GND GND GND GND N_CS"
- board text removed: "STEP DIR ENABLE GND BOOST FAULT"
- board text removed: "V1"
