File: PCB_SRT/PCB_SRT/PCB_SRT.kicad_sch (KiCad schematic)
At the start: 8 parts, among them U1 Power_header, U2 Stepper_header, U3 ESP32, U4 Stepper_header, U5 RX_TX_header, U6 Encoder_header, U7 Encoder_header, U8 RX_TX_header

Commit message: finish PCB
Parts:
- U6, U7: footprint Connector_PinHeader_2.54mm:PinHeader_1x10_P2.54mm_Vertical -> Connector_PinHeader_2.54mm:PinHeader_1x08_P2.54mm_Vertical
Connections:
- net +5V: now also U6.1 (VCC), U7.1 (VCC); no longer U6.3 (VCC), U7.3 (VCC)
- net GND: now also U2.6 (GND), U4.6 (GND), U6.3 (GND), U7.3 (GND); no longer U2.4 (GND), U4.4 (GND), U6.5 (GND), U6.6 (GND), U6.9 (unconnected), U7.5 (GND), U7.6 (GND), U7.9 (unconnected)
- net MISO: now also U6.4 (MISO), U7.4 (MISO); no longer U6.1 (MISO), U7.1 (MISO)
- net N_CS_1: now also U6.6 (N_CS); no longer U6.10 (N_CS)
- net N_CS_2: now also U7.6 (N_CS); no longer U7.10 (N_CS)
- net SCK: now also U6.5 (CLK), U7.5 (CLK); no longer U6.4 (SCK), U7.4 (SCK)
- net at U3.15 (P15): now also U4.4 (BOOST); no longer U4.5 (BOOST)
- net at U3.26 (P14): now also U4.5 (FAULT); no longer U4.6 (FAULT)
- net at U3.27 (P27): now also U2.5 (FAULT); no longer U2.6 (FAULT)
- net at U3.28 (P26): now also U2.4 (BOOST); no longer U2.5 (BOOST)
